File: pcieduino.sch (KiCad schematic (older format))
At the start: 31 parts, among them IC1 ATMEGA328P-A, J1 PCIE-MINI, J2 ANALOG_POWER, J3 ISP, J4 DIGITAL, SW1 SW_PUSH, U1 MCP2200, X1 12MHz, X2 8MHz

Commit message: progres on 01/05: mostly crystal work
Parts:
- removed X1: 12MHz, ~, symbol CRYSTAL
- removed X2: 8MHz, ~, symbol CRYSTAL
- added X1: 12MHZ, ~, symbol CRYSTAL_SMD
- added X2: 8MHz, ~, symbol CRYSTAL_SMD
Connections:
- wire segments 91 -> 95

Commit message: ATmega32U4 version work in progress
Parts:
- removed C2: 10p, ~, symbol C
- removed C8: 0.1u, ~, symbol C
- removed IC1: ATMEGA328P-A, TQFP32, symbol ATMEGA328P-A
- removed R5, R6: 1K, SM0603_Resistor, symbol R
- removed U1: MCP2200, symbol MCP2200
- removed X1: 12MHZ, ~, symbol CRYSTAL_SMD
- added C6: 1u, SM0603_Capa, symbol C
- added R1: 22, ~, symbol R
- added U1: ATMEGA32U4-AU, ~, symbol ATMEGA32U4-AU
- C1: value 10p -> 0.1u; footprint ~ -> SM0603_Capa
- C3: renamed from C7; footprint ~ -> SM0603_Capa
- C4: renamed from C9; footprint ~ -> SM0603_Capa
- C7: renamed from C5; footprint ~ -> SM0603_Capa
- C8: renamed from C4; footprint ~ -> SM0603_Capa
- R2: value R -> 22
- renumbered C6 to C2, C3 to C5, J3 to J2, J4 to J3, J2 to J4, R7 to R3, R1 to R4, R3 to R5, R4 to R6, X2 to X1
Connections:
- net labels added: D+, D-, D0/RXI, D1/TXO, D11, D12, D13, D2/SDA, D3/SCL, MISO, MOSI, RXLED, SCK, TXLED, UVCC
- net labels removed: A6, A7, D11/MOSI, D12/MISO, D13/SCK, D2, D3, DTR, RXI, TXO, USB_M, USB_P
- wire segments 95 -> 82
- no-connect marks 44 -> 37
Other:
- note added: "Input mini-PCIe connector"
- note added: "Output connectors"
- note added: "Released under Creative Commons Attribution - Share Alike CC-BY-SA 3.0 license\nBased on designs from http://arduino.cc and http://www.sparkfun.com (Pro Micro)"
- note removed: "MCP2200 Section is based on\nhttp://blog.stevemarple.co.uk/2013/01/uart-usb-converter-for-mixed-33v5v.html"
- note removed: "Released under Creative Commons Attribution - Share Alike CC-BY-SA 3.0 license\nBased on designs from http://arduino.cc"
- moved on the sheet: C2, C3, C4, C5, C7, C8, D1, D2, D3, F1, J1, J2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

Commit message: updates to the schematic (simplifications, labels, power LED
Parts:
- added D4: LED, ~, symbol LED
- added R7: 550, ~, symbol R
Connections:
- wire segments 82 -> 79
Other:
- note added: "(VIN)"
- note added: "Power LED"
- moved on the sheet: D3, R6
Changed lines of the file:
@@
-	1    0    0    -1
-$EndComp
-$Comp
-L GND #PWR08
-U 1 1 53F9FDA8
-P 10650 6200
-F 0 "#PWR08" H 10650 6200 30  0001 C CNN
-F 1 "GND" H 10650 6130 30  0001 C CNN
-F 2 "" H 10650 6200 60  0000 C CNN
-F 3 "" H 10650 6200 60  0000 C CNN
-	1    10650 6200
 	1    0    0    -1
 $EndComp
@@
 Text Label 10450 5950 0    60   ~ 0
 MOSI
-$Comp
-L VCC #PWR09
-U 1 1 53F9FDFE
-P 10600 5650
-F 0 "#PWR09" H 10600 5750 30  0001 C CNN
-F 1 "VCC" H 10600 5750 30  0000 C CNN
-F 2 "" H 10600 5650 60  0000 C CNN
-F 3 "" H 10600 5650 60  0000 C CNN
-	1    10600 5650
-	1    0    0    -1
-$EndComp
 Text Label 9650 6050 2    60   ~ 0
 RESET
-$Comp
-L VCC #PWR010
-U 1 1 53F9FFE8
-P 2750 4750
-F 0 "#PWR010" H 2750 4850 30  0001 C CNN
-F 1 "VCC" H 2750 4850 30  0000 C CNN
-F 2 "" H 2750 4750 60  0000 C CNN
-F 3 "" H 2750 4750 60  0000 C CNN
-	1    2750 4750
-	1    0    0    -1
-$EndComp
-$Comp
-L VCC #PWR011
-U 1 1 53F9FFF7
-P 3050 4750
-F 0 "#PWR011" H 3050 4850 30  0001 C CNN
-F 1 "VCC" H 3050 4850 30  0000 C CNN
-F 2 "" H 3050 4750 60  0000 C CNN
-F 3 "" H 3050 4750 60  0000 C CNN
-	1    3050 4750
-	1    0    0    -1
-$EndComp
 $Comp
 L C C3
@@
 $EndComp
 $Comp
-L GND #PWR012
+L GND #PWR08
 U 1 1 53FA004C
 P 2750 5250
-F 0 "#PWR012" H 2750 5250 30  0001 C CNN
+F 0 "#PWR08" H 2750 5250 30  0001 C CNN
 F 1 "GND" H 2750 5180 30  0001 C CNN
 F 2 "" H 2750 5250 60  0000 C CNN
@@
 $EndComp
 $Comp
-L GND #PWR013
+L GND #PWR09
 U 1 1 53FA005B
 P 3050 5250
-F 0 "#PWR013" H 3050 5250 30  0001 C CNN
+F 0 "#PWR09" H 3050 5250 30  0001 C CNN
 F 1 "GND" H 3050 5180 30  0001 C CNN
 F 2 "" H 3050 5250 60  0000 C CNN
@@
 Text Label 10150 2350 2    60   ~ 0
 D12
-$Comp
-L GND #PWR014
-U 1 1 53FA0D4F
-P 9850 2850
-F 0 "#PWR014" H 9850 2850 30  0001 C CNN
-F 1 "GND" H 9850 2780 30  0001 C CNN
-F 2 "" H 9850 2850 60  0000 C CNN
-F 3 "" H 9850 2850 60  0000 C CNN
-	1    9850 2850
-	1    0    0    -1
-$EndComp
 Text Label 10150 2550 2    60   ~ 0
 GND
@@
 L R R6
 U 1 1 53FA0DC3
-P 9550 2700
-F 0 "R6" V 9630 2700 40  0000 C CNN
-F 1 "100" V 9557 2701 40  0000 C CNN
-F 2 "SM0603_Resistor" V 9480 2700 30  0000 C CNN
-F 3 "~" H 9550 2700 30  0000 C CNN
-	1    9550 2700
+P 9800 2700
+F 0 "R6" V 9880 2700 40  0000 C CNN
+F 1 "100" V 9807 2701 40  0000 C CNN
+F 2 "SM0603_Resistor" V 9730 2700 30  0000 C CNN
+F 3 "~" H 9800 2700 30  0000 C CNN
+	1    9800 2700
 	1    0    0    -1
 $EndComp
@@
 L LED D3
 U 1 1 53FA0DD2
-P 9550 3250
-F 0 "D3" H 9550 3350 50  0000 C CNN
-F 1 "LED" H 9550 3150 50  0000 C CNN
-F 2 "~" H 9550 3250 60  0000 C CNN
-F 3 "~" H 9550 3250 60  0000 C CNN
-F 4 "LB Q39G-L2N2-35-1" H 9550 3250 60  0001 C CNN "P/N"
-	1    9550 3250
+P 9800 3250
+F 0 "D3" H 9800 3350 50  0000 C CNN
+F 1 "LED" H 9800 3150 50  0000 C CNN
+F 2 "~" H 9800 3250 60  0000 C CNN
+F 3 "~" H 9800 3250 60  0000 C CNN
+F 4 "LB Q39G-L2N2-35-1" H 9800 3250 60  0001 C CNN "P/N"
+	1    9800 3250
 	0    1    1    0
 $EndComp
 $Comp
-L GND #PWR015
+L GND #PWR010
 U 1 1 53FA0DE1
-P 9550 3550
-F 0 "#PWR015" H 9550 3550 30  0001 C CNN
-F 1 "GND" H 9550 3480 30  0001 C CNN
-F 2 "" H 9550 3550 60  0000 C CNN
-F 3 "" H 9550 3550 60  0000 C CNN
-	1    9550 3550
-	1    0    0    -1
-$EndComp
-Text Label 9400 2450 2    60   ~ 0
+P 9800 3550
+F 0 "#PWR010" H 9800 3550 30  0001 C CNN
+F 1 "GND" H 9800 3480 30  0001 C CNN
+F 2 "" H 9800 3550 60  0000 C CNN
+F 3 "" H 9800 3550 60  0000 C CNN
+	1    9800 3550
+	1    0    0    -1
+$EndComp
+Text Label 9600 2450 2    60   ~ 0
 D13
 $Comp
@@
 $EndComp
 $Comp
-L GND #PWR016
+L GND #PWR011
 U 1 1 53FA0F93
 P 3450 5250
-F 0 "#PWR016" H 3450 5250 30  0001 C CNN
+F 0 "#PWR011" H 3450 5250 30  0001 C CNN
 F 1 "GND" H 3450 5180 30  0001 C CNN
 F 2 "" H 3450 5250 60  0000 C CNN
@@
 $EndComp
 $Comp
-L VCC #PWR017
-U 1 1 53FA0FA2
-P 3450 4750
-F 0 "#PWR017" H 3450 4850 30  0001 C CNN
-F 1 "VCC" H 3450 4850 30  0000 C CNN
-F 2 "" H 3450 4750 60  0000 C CNN
-F 3 "" H 3450 4750 60  0000 C CNN
-	1    3450 4750
-	1    0    0    -1
-$EndComp
-$Comp
-L PWR_FLAG #FLG018
+L PWR_FLAG #FLG012
 U 1 1 53FA0835
 P 3950 3750
-F 0 "#FLG018" H 3950 3845 30  0001 C CNN
+F 0 "#FLG012" H 3950 3845 30  0001 C CNN
 F 1 "PWR_FLAG" H 3950 3930 30  0000 C CNN
 F 2 "" H 3950 3750 60  0000 C CNN
@@
 $EndComp
 $Comp
-L PWR_FLAG #FLG019
+L PWR_FLAG #FLG013
 U 1 1 53FF089D
 P 3000 4050
-F 0 "#FLG019" H 3000 4145 30  0001 C CNN
+F 0 "#FLG013" H 3000 4145 30  0001 C CNN
 F 1 "PWR_FLAG" H 3000 4230 30  0000 C CNN
 F 2 "" H 3000 4050 60  0000 C CNN
@@
 $EndComp
 $Comp
-L GND #PWR020
+L GND #PWR014
 U 1 1 53FF08AC
 P 3200 4100
-F 0 "#PWR020" H 3200 4100 30  0001 C CNN
+F 0 "#PWR014" H 3200 4100 30  0001 C CNN
 F 1 "GND" H 3200 4030 30  0001 C CNN
 F 2 "" H 3200 4100 60  0000 C CNN
@@
 $EndComp
 $Comp
-L VCC #PWR021
+L VCC #PWR015
 U 1 1 549E7797
 P 7950 5950
-F 0 "#PWR021" H 7950 6050 30  0001 C CNN
+F 0 "#PWR015" H 7950 6050 30  0001 C CNN
 F 1 "VCC" H 7950 6050 30  0000 C CNN
 F 2 "" H 7950 5950 60  0000 C CNN
@@
 $EndComp
 $Comp
-L GND #PWR022
+L GND #PWR016
 U 1 1 54A7DBD9
 P 2650 6500
-F 0 "#PWR022" H 2650 6500 30  0001 C CNN
+F 0 "#PWR016" H 2650 6500 30  0001 C CNN
 F 1 "GND" H 2650 6430 30  0001 C CNN
 F 2 "" H 2650 6500 60  0000 C CNN
@@
 UVCC
 $Comp
-L GND #PWR023
+L GND #PWR017
 U 1 1 55433DE5
 P 2200 5250
-F 0 "#PWR023" H 2200 5250 30  0001 C CNN
+F 0 "#PWR017" H 2200 5250 30  0001 C CNN
 F 1 "GND" H 2200 5180 30  0001 C CNN
 F 2 "" H 2200 5250 60  0000 C CNN
@@
 D-
 $Comp
-L GND #PWR024
+L GND #PWR018
 U 1 1 554344DD
 P 5950 2350
-F 0 "#PWR024" H 5950 2350 30  0001 C CNN
+F 0 "#PWR018" H 5950 2350 30  0001 C CNN
 F 1 "GND" H 5950 2280 30  0001 C CNN
 F 2 "" H 5950 2350 60  0000 C CNN
@@
 $EndComp
 $Comp
-L GND #PWR025
+L GND #PWR019
 U 1 1 55434502
 P 5250 2650
-F 0 "#PWR025" H 5250 2650 30  0001 C CNN
+F 0 "#PWR019" H 5250 2650 30  0001 C CNN
 F 1 "GND" H 5250 2580 30  0001 C CNN
 F 2 "" H 5250 2650 60  0000 C CNN
@@
 D12
 $Comp
-L GND #PWR026
+L GND #PWR020
 U 1 1 5543599F
 P 8850 3400
-F 0 "#PWR026" H 8850 3400 30  0001 C CNN
+F 0 "#PWR020" H 8850 3400 30  0001 C CNN
 F 1 "GND" H 8850 3330 30  0001 C CNN
 F 2 "" H 8850 3400 60  0000 C CNN
@@
 Text Label 8100 4700 0    60   ~ 0
 RXLED
+Text Notes 9150 850  0    60   ~ 0
+Output connectors
+Text Notes 1300 950  0    60   ~ 0
+Input mini-PCIe connector
+$Comp
+L LED D4
+U 1 1 5543889F
+P 3950 5000
+F 0 "D4" H 3950 5100 50  0000 C CNN
+F 1 "LED" H 3950 4900 50  0000 C CNN
+F 2 "~" H 3950 5000 60  0000 C CNN
+F 3 "~" H 3950 5000 60  0000 C CNN
+	1    3950 5000
+	0    1    1    0
+$EndComp
+$Comp
+L R R7
+U 1 1 554389A4
+P 3950 5500
+F 0 "R7" V 4030 5500 40  0000 C CNN
+F 1 "550" V 3957 5501 40  0000 C CNN
+F 2 "~" V 3880 5500 30  0000 C CNN
+F 3 "~" H 3950 5500 30  0000 C CNN
+	1    3950 5500
+	1    0    0    -1
+$EndComp
+$Comp
+L GND #PWR021
+U 1 1 55438B10
+P 3950 5800
+F 0 "#PWR021" H 3950 5800 30  0001 C CNN
+F 1 "GND" H 3950 5730 30  0001 C CNN
+F 2 "" H 3950 5800 60  0000 C CNN
+F 3 "" H 3950 5800 60  0000 C CNN
+	1    3950 5800
+	1    0    0    -1
+$EndComp
 Wire Wire Line
 	5050 3250 5050 3550
@@
 Wire Wire Line
 	3450 5200 3450 5250
-Wire Wire Line
-	3450 4800 3450 4750
-Connection ~ 9550 2450
-Wire Wire Line
-	9400 2450 10150 2450
-Wire Wire Line
-	9550 3050 9550 2950
-Wire Wire Line
-	9550 3550 9550 3450
-Wire Wire Line
-	9850 2550 10150 2550
-Wire Wire Line
-	9850 2850 9850 2550
-Wire Wire Line
-	3050 4800 3050 4750
-Wire Wire Line
-	2750 4800 2750 4750
+Connection ~ 9800 2450
+Wire Wire Line
+	9800 3050 9800 2950
+Wire Wire Line
+	9800 3550 9800 3450
 Wire Wire Line
 	3050 5200 3050 5250
 Wire Wire Line
 	2750 5200 2750 5250
-Wire Wire Line
-	10600 5850 10600 5650
-Wire Wire Line
-	10450 5850 10600 5850
-Wire Wire Line
-	10650 6050 10650 6200
-Wire Wire Line
-	10450 6050 10650 6050
 Wire Wire Line
 	3900 3750 4150 3750
@@
 Wire Notes Line
 	9100 6400 9100 900
-Text Notes 9150 850  0    60   ~ 0
-Output connectors
-Text Notes 1300 950  0    60   ~ 0
-Input mini-PCIe connector
+Wire Wire Line
+	3950 5200 3950 5250
+Wire Wire Line
+	3950 5750 3950 5800
+Wire Wire Line
+	3950 4800 3950 4750
+$Comp
+L VCC #PWR022
+U 1 1 554388AE
+P 3950 4750
+F 0 "#PWR022" H 3950 4850 30  0001 C CNN
+F 1 "VCC" H 3950 4850 30  0000 C CNN
+F 2 "" H 3950 4750 60  0000 C CNN
+F 3 "" H 3950 4750 60  0000 C CNN
+	1    3950 4750
+	1    0    0    -1
+$EndComp
+Wire Wire Line
+	3450 4800 3450 4750
+$Comp
+L VCC #PWR023
+U 1 1 53FA0FA2
+P 3450 4750
+F 0 "#PWR023" H 3450 4850 30  0001 C CNN
+F 1 "VCC" H 3450 4850 30  0000 C CNN
+F 2 "" H 3450 4750 60  0000 C CNN
+F 3 "" H 3450 4750 60  0000 C CNN
+	1    3450 4750
+	1    0    0    -1
+$EndComp
+Wire Wire Line
+	3050 4800 3050 4750
+$Comp
+L VCC #PWR024
+U 1 1 53F9FFF7
+P 3050 4750
+F 0 "#PWR024" H 3050 4850 30  0001 C CNN
+F 1 "VCC" H 3050 4850 30  0000 C CNN
+F 2 "" H 3050 4750 60  0000 C CNN
+F 3 "" H 3050 4750 60  0000 C CNN
+	1    3050 4750
+	1    0    0    -1
+$EndComp
+Wire Wire Line
+	2750 4800 2750 4750
+$Comp
+L VCC #PWR025
+U 1 1 53F9FFE8
+P 2750 4750
+F 0 "#PWR025" H 2750 4850 30  0001 C CNN
+F 1 "VCC" H 2750 4850 30  0000 C CNN
+F 2 "" H 2750 4750 60  0000 C CNN
+F 3 "" H 2750 4750 60  0000 C CNN
+	1    2750 4750
+	1    0    0    -1
+$EndComp
+Text Notes 4050 5200 0    60   ~ 0
+Power LED
+Text Label 10450 6050 0    60   ~ 0
+GND
+Text Label 10450 5850 0    60   ~ 0
+VCC
+Text Label 3200 4050 2    60   ~ 0
+GND
+Wire Wire Line
+	10150 2450 9600 2450
+Text Notes 9650 4550 0    60   ~ 0
+(VIN)
 $EndSCHEMATC

Commit message: work in progress: Mouser part numbers, new switch footprint, fixed footprint mixups
Parts:
- C1, C3, C4: MouserPN (none) -> 581-060316C104K
- C2: footprint ~ -> SM1206Pol; MouserPN (none) -> 647-F931A106KAA
- C5: MouserPN (none) -> 581-060316C104K; Seed PN 0100020P1 -> (none)
- C6: MouserPN (none) -> 581-0603YC105KAT2A
- C7, C8: MouserPN (none) -> 81-GRM0335C1H100FA1D
- D1, D3: footprint ~ -> LED-0603
- D2: footprint ~ -> LED-0603; MouserPN (none) -> 720-LOL29KH2L124Z
- D4: footprint ~ -> LED-0603; MouserPN (none) -> 720-LSL29K-G1H2-1-Z
- F1: MouserPN (none) -> 576-1206L110THYR
- R1, R2: footprint ~ -> SM0603_Resistor; MouserPN (none) -> 71-CRCW0603-22-E3
- R3: MouserPN (none) -> 71-CRCW0603-10K-E3
- R4, R5, R7: value 550 -> 549; footprint ~ -> SM0603_Resistor; MouserPN (none) -> 71-CRCW0603-549-E3
- R6: MouserPN (none) -> 71-CRCW0603-100-E3
- SW1: MouserPN (none) -> 612-TL3313AF100QG
- U1: footprint ~ -> TQFP44; MouserP# (none) -> 556-ATMEGA32U4-AU
- X1: MouserPN (none) -> 815-ABM3B-8.0-10-1UT
Other:
- note added: "Blue"
- note added: "Green"
- note added: "Orange"
- note added: "Power LED\nRed"
- note removed: "Power LED"
Changed lines of the file:
@@
 Sheet 1 1
 Title "PCIeDuino32u4 v1"
-Date "1 may 2015"
+Date "2 may 2015"
 Rev "1"
 Comp "moonpunch.org"
@@
 F 0 "C8" H 5500 3650 40  0000 L CNN
 F 1 "10p" H 5506 3465 40  0000 L CNN
-F 2 "SM0603_Capa" H 5538 3400 30  0000 C CNN
+F 2 "SM0603_Capa" H 5538 3400 30  0001 C CNN
 F 3 "~" H 5500 3550 60  0000 C CNN
+F 4 "81-GRM0335C1H100FA1D" H 5500 3550 60  0001 C CNN "MouserPN"
 	1    5500 3550
 	0    1    1    0
@@
 F 0 "C7" H 5500 3050 40  0000 L CNN
 F 1 "10p" H 5506 2865 40  0000 L CNN
-F 2 "SM0603_Capa" H 5538 2800 30  0000 C CNN
+F 2 "SM0603_Capa" H 5538 2800 30  0001 C CNN
 F 3 "~" H 5500 2950 60  0000 C CNN
+F 4 "81-GRM0335C1H100FA1D" H 5500 2950 60  0001 C CNN "MouserPN"
 	1    5500 2950
 	0    1    1    0
@@
 F 0 "R3" V 4830 2500 40  0000 C CNN
 F 1 "10K" V 4757 2501 40  0000 C CNN
-F 2 "SM0603_Resistor" V 4680 2500 30  0000 C CNN
+F 2 "SM0603_Resistor" V 4680 2500 30  0001 C CNN
 F 3 "~" H 4750 2500 30  0000 C CNN
+F 4 "71-CRCW0603-10K-E3" V 4750 2500 60  0001 C CNN "MouserPN"
 	1    4750 2500
 	1    0    0    -1
@@
 F 1 "SW_PUSH" H 4750 3070 50  0000 C CNN
 F 2 "~" H 4750 3150 60  0000 C CNN
-F 3 "~" H 4750 3150 60  0000 C CNN
+F 3 "http://www.mouser.com/ds/2/140/TL3313-346065.pdf" H 4750 3150 60  0001 C CNN
+F 4 "612-TL3313AF100QG" H 4750 3150 60  0001 C CNN "MouserPN"
 	1    4750 3150
 	0    -1   -1   0
@@
 F 0 "C5" H 5250 1900 40  0000 L CNN
 F 1 "0.1u" H 5256 1715 40  0000 L CNN
-F 2 "SM0603_Capa" H 5288 1650 30  0000 C CNN
+F 2 "SM0603_Capa" H 5288 1650 30  0001 C CNN
 F 3 "~" H 5250 1800 60  0000 C CNN
-F 4 "0100020P1" H 5250 1800 60  0001 C CNN "Seed PN"
+F 4 "581-060316C104K" H 5250 1800 60  0001 C CNN "MouserPN"
 	1    5250 1800
 	1    0    0    -1
@@
 F 2 "~" H 3650 3750 60  0000 C CNN
 F 3 "~" H 3650 3750 60  0000 C CNN
+F 4 "576-1206L110THYR" H 3650 3750 60  0001 C CNN "MouserPN"
 	1    3650 3750
 	1    0    0    -1
@@
 F 0 "C3" H 3050 5100 40  0000 L CNN
 F 1 "0.1u" H 3056 4915 40  0000 L CNN
-F 2 "SM0603_Capa" H 3088 4850 30  0000 C CNN
+F 2 "SM0603_Capa" H 3088 4850 30  0001 C CNN
 F 3 "~" H 3050 5000 60  0000 C CNN
+F 4 "581-060316C104K" H 3050 5000 60  0001 C CNN "MouserPN"
 	1    3050 5000
 	1    0    0    -1
@@
 F 0 "C2" H 2800 5100 50  0000 L CNN
 F 1 "10u" H 2800 4900 50  0000 L CNN
-F 2 "~" H 2750 5000 60  0000 C CNN
+F 2 "SM1206Pol" H 2750 5000 60  0001 C CNN
 F 3 "~" H 2750 5000 60  0000 C CNN
+F 4 "647-F931A106KAA" H 2750 5000 60  0001 C CNN "MouserPN"
 	1    2750 5000
 	1    0    0    -1
@@
 F 0 "R6" V 9880 2700 40  0000 C CNN
 F 1 "100" V 9807 2701 40  0000 C CNN
-F 2 "SM0603_Resistor" V 9730 2700 30  0000 C CNN
+F 2 "SM0603_Resistor" V 9730 2700 30  0001 C CNN
 F 3 "~" H 9800 2700 30  0000 C CNN
+F 4 "71-CRCW0603-100-E3" V 9800 2700 60  0001 C CNN "MouserPN"
 	1    9800 2700
 	1    0    0    -1
@@
 F 0 "D3" H 9800 3350 50  0000 C CNN
 F 1 "LED" H 9800 3150 50  0000 C CNN
-F 2 "~" H 9800 3250 60  0000 C CNN
+F 2 "LED-0603" H 9800 3250 60  0001 C CNN
 F 3 "~" H 9800 3250 60  0000 C CNN
 F 4 "LB Q39G-L2N2-35-1" H 9800 3250 60  0001 C CNN "P/N"
@@
 F 0 "C4" H 3450 5100 40  0000 L CNN
 F 1 "0.1u" H 3456 4915 40  0000 L CNN
-F 2 "SM0603_Capa" H 3488 4850 30  0000 C CNN
+F 2 "SM0603_Capa" H 3488 4850 30  0001 C CNN
 F 3 "~" H 3450 5000 60  0000 C CNN
+F 4 "581-060316C104K" H 3450 5000 60  0001 C CNN "MouserPN"
 	1    3450 5000
 	1    0    0    -1
@@
 F 0 "D1" H 7800 5100 50  0000 C CNN
 F 1 "LED" H 7800 4900 50  0000 C CNN
-F 2 "~" H 7800 5000 60  0000 C CNN
+F 2 "LED-0603" H 7800 5000 60  0001 C CNN
 F 3 "~" H 7800 5000 60  0000 C CNN
 F 4 "LS L29K-G1H2-1-Z" H 7800 5000 60  0001 C CNN "P/N"
@@
 F 0 "D2" H 8100 5100 50  0000 C CNN
 F 1 "LED" H 8100 4900 50  0000 C CNN
-F 2 "~" H 8100 5000 60  0000 C CNN
+F 2 "LED-0603" H 8100 5000 60  0001 C CNN
 F 3 "~" H 8100 5000 60  0000 C CNN
+F 4 "720-LOL29KH2L124Z" H 8100 5000 60  0001 C CNN "MouserPN"
 	1    8100 5000
 	0    -1   -1   0
@@
 P 7800 5550
 F 0 "R4" V 7880 5550 40  0000 C CNN
-F 1 "550" V 7807 5551 40  0000 C CNN
-F 2 "~" V 7730 5550 30  0000 C CNN
+F 1 "549" V 7807 5551 40  0000 C CNN
+F 2 "SM0603_Resistor" V 7730 5550 30  0001 C CNN
 F 3 "~" H 7800 5550 30  0000 C CNN
+F 4 "71-CRCW0603-549-E3" V 7800 5550 60  0001 C CNN "MouserPN"
 	1    7800 5550
 	1    0    0    -1
@@
 P 8100 5550
 F 0 "R5" V 8180 5550 40  0000 C CNN
-F 1 "550" V 8107 5551 40  0000 C CNN
-F 2 "~" V 8030 5550 30  0000 C CNN
+F 1 "549" V 8107 5551 40  0000 C CNN
+F 2 "SM0603_Resistor" V 8030 5550 30  0001 C CNN
 F 3 "~" H 8100 5550 30  0000 C CNN
+F 4 "71-CRCW0603-549-E3" V 8100 5550 60  0001 C CNN "MouserPN"
 	1    8100 5550
 	1    0    0    -1
@@
 F 2 "~" H 5800 3250 60  0000 C CNN
 F 3 "~" H 5800 3250 60  0000 C CNN
+F 4 "815-ABM3B-8.0-10-1UT" H 5800 3250 60  0001 C CNN "MouserPN"
 	1    5800 3250
 	0    1    1    0
@@
 F 0 "U1" H 6400 4450 60  0000 C CNN
 F 1 "ATMEGA32U4-AU" H 6650 1200 60  0000 C CNN
-F 2 "~" H 8500 3850 60  0000 C CNN
+F 2 "TQFP44" H 8500 3850 60  0001 C CNN
 F 3 "~" H 8500 3850 60  0000 C CNN
+F 4 "556-ATMEGA32U4-AU" H 7300 2750 60  0001 C CNN "MouserP#"
 	1    7300 2750
 	1    0    0    -1
@@
 F 0 "C1" H 2200 5100 40  0000 L CNN
 F 1 "0.1u" H 2206 4915 40  0000 L CNN
-F 2 "SM0603_Capa" H 2200 4850 30  0000 C CNN
+F 2 "SM0603_Capa" H 2200 4850 30  0001 C CNN
 F 3 "~" H 2200 5000 60  0000 C CNN
+F 4 "581-060316C104K" H 2200 5000 60  0001 C CNN "MouserPN"
 	1    2200 5000
 	1    0    0    -1
@@
 F 0 "C6" H 5250 2500 40  0000 L CNN
 F 1 "1u" H 5256 2315 40  0000 L CNN
-F 2 "SM0603_Capa" H 5288 2250 30  0000 C CNN
+F 2 "SM0603_Capa" H 5288 2250 30  0001 C CNN
 F 3 "~" H 5250 2400 60  0000 C CNN
+F 4 "581-0603YC105KAT2A" H 5250 2400 60  0001 C CNN "MouserPN"
 	1    5250 2400
 	1    0    0    -1
@@
 F 0 "R2" V 3730 3050 40  0000 C CNN
 F 1 "22" V 3657 3051 40  0000 C CNN
-F 2 "~" V 3580 3050 30  0000 C CNN
+F 2 "SM0603_Resistor" V 3580 3050 30  0001 C CNN
 F 3 "~" H 3650 3050 30  0000 C CNN
+F 4 "71-CRCW0603-22-E3" V 3650 3050 60  0001 C CNN "MouserPN"
 	1    3650 3050
 	0    1    1    0
@@
 F 0 "R1" V 3730 2950 40  0000 C CNN
 F 1 "22" V 3657 2951 40  0000 C CNN
-F 2 "~" V 3580 2950 30  0000 C CNN
+F 2 "SM0603_Resistor" V 3580 2950 30  0001 C CNN
 F 3 "~" H 3650 2950 30  0000 C CNN
+F 4 "71-CRCW0603-22-E3" V 3650 2950 60  0001 C CNN "MouserPN"
 	1    3650 2950
 	0    -1   -1   0
@@
 F 0 "D4" H 3950 5100 50  0000 C CNN
 F 1 "LED" H 3950 4900 50  0000 C CNN
-F 2 "~" H 3950 5000 60  0000 C CNN
+F 2 "LED-0603" H 3950 5000 60  0001 C CNN
 F 3 "~" H 3950 5000 60  0000 C CNN
+F 4 "720-LSL29K-G1H2-1-Z" H 3950 5000 60  0001 C CNN "MouserPN"
 	1    3950 5000
 	0    1    1    0
@@
 P 3950 5500
 F 0 "R7" V 4030 5500 40  0000 C CNN
-F 1 "550" V 3957 5501 40  0000 C CNN
-F 2 "~" V 3880 5500 30  0000 C CNN
+F 1 "549" V 3957 5501 40  0000 C CNN
+F 2 "SM0603_Resistor" V 3880 5500 30  0001 C CNN
 F 3 "~" H 3950 5500 30  0000 C CNN
+F 4 "71-CRCW0603-549-E3" V 3950 5500 60  0001 C CNN "MouserPN"
 	1    3950 5500
 	1    0    0    -1
@@
 $EndComp
 Text Notes 4050 5200 0    60   ~ 0
-Power LED
+Power LED\nRed
 Text Label 10450 6050 0    60   ~ 0
 GND
@@
 Text Notes 9650 4550 0    60   ~ 0
 (VIN)
+Text Notes 7650 4900 2    60   ~ 0
+Green
+Text Notes 8250 4900 0    60   ~ 0
+Orange
+Text Notes 9900 3450 0    60   ~ 0
+Blue
 $EndSCHEMATC

Commit message: work in progress, after autorouting and all connections
Changed lines of the file:
@@
 Sheet 1 1
 Title "PCIeDuino32u4 v1"
-Date "2 may 2015"
+Date "3 may 2015"
 Rev "1"
 Comp "moonpunch.org"
@@
 U 1 1 55435189
 P 3650 2950
-F 0 "R1" V 3730 2950 40  0000 C CNN
+F 0 "R1" V 3550 2950 40  0000 C CNN
 F 1 "22" V 3657 2951 40  0000 C CNN
 F 2 "SM0603_Resistor" V 3580 2950 30  0001 C CNN
@@
 F 4 "71-CRCW0603-22-E3" V 3650 2950 60  0001 C CNN "MouserPN"
 	1    3650 2950
-	0    -1   -1   0
+	0    1    1    0
 $EndComp
 Text Label 3900 2950 0    60   ~ 0
