File: pcieduino.sch (KiCad schematic (older format))
At the start: 29 parts, among them J1 PCIE-MINI, J2 ISP, J3 DIGITAL, J4 ANALOG_POWER, SW1 SW_PUSH, U1 ATMEGA32U4-AU, X1 8MHz

Commit message: Updated version, ready to print
* fixed XTAL footprint
* changed 10u bypass footprint
* general layout improvements
* added Moonpunch logo
Parts:
- removed C2: 10u, SM1206Pol, symbol CP1
- added C2: 10u, ~, symbol C
- C7, C8: MouserPN 81-GRM0335C1H100FA1D -> 581-06035A100J
- D1: value LED -> TX
- D2: value LED -> RX
- D3: value LED -> D13
- D4: value LED -> PWR
- SW1: value SW_PUSH -> Reset
- U1: value ATMEGA32U4-AU -> ATMEGA32U4
- X1: footprint ~ -> SMDXTAL_50x32
Other:
- note added: "(-AU)"
Changed lines of the file:
@@
 Sheet 1 1
 Title "PCIeDuino32u4 v1"
-Date "3 may 2015"
+Date "24 may 2015"
 Rev "1"
 Comp "moonpunch.org"
@@
 F 2 "SM0603_Capa" H 5538 3400 30  0001 C CNN
 F 3 "~" H 5500 3550 60  0000 C CNN
-F 4 "81-GRM0335C1H100FA1D" H 5500 3550 60  0001 C CNN "MouserPN"
+F 4 "581-06035A100J" H 5500 3550 60  0001 C CNN "MouserPN"
 	1    5500 3550
 	0    1    1    0
@@
 F 2 "SM0603_Capa" H 5538 2800 30  0001 C CNN
 F 3 "~" H 5500 2950 60  0000 C CNN
-F 4 "81-GRM0335C1H100FA1D" H 5500 2950 60  0001 C CNN "MouserPN"
+F 4 "581-06035A100J" H 5500 2950 60  0001 C CNN "MouserPN"
 	1    5500 2950
 	0    1    1    0
@@
 P 4750 3150
 F 0 "SW1" H 4900 3260 50  0000 C CNN
-F 1 "SW_PUSH" H 4750 3070 50  0000 C CNN
+F 1 "Reset" H 4750 3070 50  0000 C CNN
 F 2 "~" H 4750 3150 60  0000 C CNN
 F 3 "http://www.mouser.com/ds/2/140/TL3313-346065.pdf" H 4750 3150 60  0001 C CNN
@@
 	1    0    0    -1
 $EndComp
-$Comp
-L CP1 C2
-U 1 1 53FA01C2
-P 2750 5000
-F 0 "C2" H 2800 5100 50  0000 L CNN
-F 1 "10u" H 2800 4900 50  0000 L CNN
-F 2 "SM1206Pol" H 2750 5000 60  0001 C CNN
-F 3 "~" H 2750 5000 60  0000 C CNN
-F 4 "647-F931A106KAA" H 2750 5000 60  0001 C CNN "MouserPN"
-	1    2750 5000
-	1    0    0    -1
-$EndComp
 Text Label 10150 4850 2    60   ~ 0
 VCC
@@
 P 9800 3250
 F 0 "D3" H 9800 3350 50  0000 C CNN
-F 1 "LED" H 9800 3150 50  0000 C CNN
+F 1 "D13" H 9800 3150 50  0000 C CNN
 F 2 "LED-0603" H 9800 3250 60  0001 C CNN
 F 3 "~" H 9800 3250 60  0000 C CNN
@@
 P 7800 5000
 F 0 "D1" H 7800 5100 50  0000 C CNN
-F 1 "LED" H 7800 4900 50  0000 C CNN
+F 1 "TX" H 7800 4900 50  0000 C CNN
 F 2 "LED-0603" H 7800 5000 60  0001 C CNN
 F 3 "~" H 7800 5000 60  0000 C CNN
@@
 P 8100 5000
 F 0 "D2" H 8100 5100 50  0000 C CNN
-F 1 "LED" H 8100 4900 50  0000 C CNN
+F 1 "RX" H 8100 4900 50  0000 C CNN
 F 2 "LED-0603" H 8100 5000 60  0001 C CNN
 F 3 "~" H 8100 5000 60  0000 C CNN
@@
 F 0 "X1" H 5800 3340 30  0000 C CNN
 F 1 "8MHz" H 5830 3140 30  0000 L CNN
-F 2 "~" H 5800 3250 60  0000 C CNN
+F 2 "SMDXTAL_50x32" H 5800 3250 60  0001 C CNN
 F 3 "~" H 5800 3250 60  0000 C CNN
 F 4 "815-ABM3B-8.0-10-1UT" H 5800 3250 60  0001 C CNN "MouserPN"
@@
 P 7300 2750
 F 0 "U1" H 6400 4450 60  0000 C CNN
-F 1 "ATMEGA32U4-AU" H 6650 1200 60  0000 C CNN
+F 1 "ATMEGA32U4" H 6650 1200 60  0000 C CNN
 F 2 "TQFP44" H 8500 3850 60  0001 C CNN
 F 3 "~" H 8500 3850 60  0000 C CNN
@@
 P 3950 5000
 F 0 "D4" H 3950 5100 50  0000 C CNN
-F 1 "LED" H 3950 4900 50  0000 C CNN
+F 1 "PWR" H 3950 4900 50  0000 C CNN
 F 2 "LED-0603" H 3950 5000 60  0001 C CNN
 F 3 "~" H 3950 5000 60  0000 C CNN
@@
 Text Notes 9900 3450 0    60   ~ 0
 Blue
+$Comp
+L C C2
+U 1 1 5560A72B
+P 2750 5000
+F 0 "C2" H 2750 5100 40  0000 L CNN
+F 1 "10u" H 2756 4915 40  0000 L CNN
+F 2 "~" H 2788 4850 30  0000 C CNN
+F 3 "~" H 2750 5000 60  0000 C CNN
+F 4 "581-0805YD106K" H 2750 5000 60  0001 C CNN "Mouser PN"
+	1    2750 5000
+	1    0    0    -1
+$EndComp
+Text Notes 7000 4350 0    60   ~ 0
+(-AU)
 $EndSCHEMATC
